Commit message: Transfer & Rebase Updates to MS210 Support package

File: motoman/motoman_ms210_support/urdf/ms210.xacro (robot description, xacro)
@@ -1,10 +1,5 @@
 <?xml version="1.0" ?>
 <robot name="motoman_ms210" xmlns:xacro="http://ros.org/wiki/xacro">
-	<!-- Properties -->
-	<material name="yaskawa_blue">
-		<color rgba="0.12941 0.14902 0.74902 1" />
-	</material>
-	<!-- Robot -->
-	<xacro:include filename="$(find motoman_ms210_support)/urdf/ms210_macro.xacro" />
-	<xacro:motoman_ms210 prefix=""/>
+  <xacro:include filename="$(find motoman_ms210_support)/urdf/ms210_macro.xacro" />
+  <xacro:motoman_ms210 prefix=""/>
 </robot>

File: motoman/motoman_ms210_support/urdf/ms210_macro.xacro (robot description, xacro)
@@ -2,21 +2,21 @@
 <robot xmlns:xacro="http://ros.org/wiki/xacro">
 <xacro:macro name="motoman_ms210" params="prefix">
+  <!-- Properties -->
+  <material name="yaskawa_blue">
+    <color rgba="0 0.35546875 0.671875 1" />
+  </material>
   <!-- link list -->
   <link  name="${prefix}base_link">
     <visual>
-      <origin
-        xyz="0 0 0"
-        rpy="0 0 0" />
+      <origin xyz="0 0 0" rpy="0 0 0" />
       <geometry>
-        <mesh filename="package://motoman_ms210_support/meshes/ms210/visual/MS210_BASE_AXIS.STL" />
+        <mesh filename="package://motoman_ms210_support/meshes/ms210/visual/base_link.stl" />
       </geometry>
       <material name="yaskawa_blue"/>
     </visual>
     <collision>
-      <origin
-        xyz="0 0 0"
-        rpy="0 0 0" />
+      <origin xyz="0 0 0" rpy="0 0 0" />
       <geometry>
-        <mesh filename="package://motoman_ms210_support/meshes/ms210/collision/MS210_BASE_AXIS.STL" />
+        <mesh filename="package://motoman_ms210_support/meshes/ms210/collision/base_link.stl" />
       </geometry>
     </collision>
@@ -24,18 +24,14 @@
   <link  name="${prefix}link_s">
     <visual>
-      <origin
-        xyz="0 0 0"
-        rpy="0 0 0" />
+      <origin xyz="0 0 0" rpy="0 0 0" />
       <geometry>
-        <mesh filename="package://motoman_ms210_support/meshes/ms210/visual/MS210_S_AXIS.STL" />
+        <mesh filename="package://motoman_ms210_support/meshes/ms210/visual/link_1_s.stl" />
       </geometry>
       <material name="yaskawa_blue"/>
     </visual>
     <collision>
-      <origin
-        xyz="0 0 0"
-        rpy="0 0 0" />
+      <origin xyz="0 0 0" rpy="0 0 0" />
       <geometry>
-        <mesh filename="package://motoman_ms210_support/meshes/ms210/collision/MS210_S_AXIS.STL" />
+        <mesh filename="package://motoman_ms210_support/meshes/ms210/collision/link_1_s.stl" />
       </geometry>
     </collision>
@@ -43,18 +39,14 @@
   <link  name="${prefix}link_l">
     <visual>
-      <origin
-        xyz="0 0 0"
-        rpy="0 0 0" />
+      <origin xyz="0 0 0" rpy="0 0 0" />
       <geometry>
-        <mesh filename="package://motoman_ms210_support/meshes/ms210/visual/MS210_L_AXIS.STL" />
+        <mesh filename="package://motoman_ms210_support/meshes/ms210/visual/link_2_l.stl" />
       </geometry>
       <material name="yaskawa_blue"/>
     </visual>
     <collision>
-      <origin
-        xyz="0 0 0"
-        rpy="0 0 0" />
+      <origin xyz="0 0 0" rpy="0 0 0" />
       <geometry>
-        <mesh filename="package://motoman_ms210_support/meshes/ms210/collision/MS210_L_AXIS.STL" />
+        <mesh filename="package://motoman_ms210_support/meshes/ms210/collision/link_2_l.stl" />
       </geometry>
     </collision>
@@ -62,18 +54,14 @@
   <link  name="${prefix}link_u">
     <visual>
-      <origin
-        xyz="0 0 0"
-        rpy="0 0 0" />
+      <origin xyz="0 0 0" rpy="0 0 0" />
       <geometry>
-        <mesh filename="package://motoman_ms210_support/meshes/ms210/visual/MS210_U_AXIS.STL" />
+        <mesh filename="package://motoman_ms210_support/meshes/ms210/visual/link_3_u.stl" />
       </geometry>
       <material name="yaskawa_blue"/>
     </visual>
     <collision>
-      <origin
-        xyz="0 0 0"
-        rpy="0 0 0" />
+      <origin xyz="0 0 0" rpy="0 0 0" />
       <geometry>
-        <mesh filename="package://motoman_ms210_support/meshes/ms210/collision/MS210_U_AXIS.STL" />
+        <mesh filename="package://motoman_ms210_support/meshes/ms210/collision/link_3_u.stl" />
       </geometry>
     </collision>
@@ -81,18 +69,14 @@
   <link  name="${prefix}link_r">
     <visual>
-      <origin
-        xyz="0 0 0"
-        rpy="0 0 0" />
+      <origin xyz="0 0 0" rpy="0 0 0" />
       <geometry>
-        <mesh filename="package://motoman_ms210_support/meshes/ms210/visual/MS210_R_AXIS.STL" />
+        <mesh filename="package://motoman_ms210_support/meshes/ms210/visual/link_4_r.stl" />
       </geometry>
       <material name="yaskawa_blue"/>
     </visual>
     <collision>
-      <origin
-        xyz="0 0 0"
-        rpy="0 0 0" />
+      <origin xyz="0 0 0" rpy="0 0 0" />
       <geometry>
-        <mesh filename="package://motoman_ms210_support/meshes/ms210/collision/MS210_R_AXIS.STL" />
+        <mesh filename="package://motoman_ms210_support/meshes/ms210/collision/link_4_r.stl" />
       </geometry>
     </collision>
@@ -100,18 +84,14 @@
   <link  name="${prefix}link_b">
     <visual>
-      <origin
-        xyz="0 0 0"
-        rpy="0 0 0" />
+      <origin xyz="0 0 0" rpy="0 0 0" />
       <geometry>
-        <mesh filename="package://motoman_ms210_support/meshes/ms210/visual/MS210_B_AXIS.STL" />
+        <mesh filename="package://motoman_ms210_support/meshes/ms210/visual/link_5_b.stl" />
       </geometry>
       <material name="yaskawa_blue"/>
     </visual>
     <collision>
-      <origin
-        xyz="0 0 0"
-        rpy="0 0 0" />
+      <origin xyz="0 0 0" rpy="0 0 0" />
       <geometry>
-        <mesh filename="package://motoman_ms210_support/meshes/ms210/collision/MS210_B_AXIS.STL" />
+        <mesh filename="package://motoman_ms210_support/meshes/ms210/collision/link_5_b.stl" />
       </geometry>
     </collision>
@@ -119,18 +99,14 @@
   <link  name="${prefix}link_t">
     <visual>
-      <origin
-        xyz="0 0 0"
-        rpy="0 0 0" />
+      <origin xyz="0 0 0" rpy="0 0 0" />
       <geometry>
-        <mesh filename="package://motoman_ms210_support/meshes/ms210/visual/MS210_T_AXIS.STL" />
+        <mesh filename="package://motoman_ms210_support/meshes/ms210/visual/link_6_t.stl" />
       </geometry>
       <material name="yaskawa_blue"/>
     </visual>
     <collision>
-      <origin
-        xyz="0 0 0"
-        rpy="0 0 0" />
+      <origin xyz="0 0 0" rpy="0 0 0" />
       <geometry>
-        <mesh filename="package://motoman_ms210_support/meshes/ms210/collision/MS210_T_AXIS.STL" />
+        <mesh filename="package://motoman_ms210_support/meshes/ms210/collision/link_6_t.stl" />
       </geometry>
     </collision>
@@ -142,73 +118,56 @@
     <parent link="${prefix}base_link" />
     <child  link="${prefix}link_s" />
-    <origin xyz="0 0 0.342" rpy="0 0 0" />
+    <origin xyz="0 0 0.650" rpy="0 0 0" />
     <axis   xyz="0 0 1" />
-    <limit
-      lower="-3.1416"
-      upper="3.1416"
-      effort="0"
-      velocity="2.09440" />
+    <limit lower="${radians(-180)}" upper="${radians(180)}" effort="6276.26" velocity="${radians(120)}" />
   </joint>
   <joint name="${prefix}joint_l" type="revolute">
     <parent link="${prefix}link_s" />
     <child link="${prefix}link_l" />
-    <origin xyz="0.325 0 0.333" rpy="0 0 0" />
+    <origin xyz="0.325 0 0" rpy="0 0 0" />
     <axis xyz="0 1 0" />
-    <limit
-      lower="-1.0472"
-      upper="1.3265"
-      effort="0"
-      velocity="1.69297" />
+    <limit lower="${radians(-60)}" upper="${radians(76)}" effort="9806.65" velocity="${radians(97)}" />
   </joint>
   <joint name="${prefix}joint_u" type="revolute">
     <parent link="${prefix}link_l" />
     <child link="${prefix}link_u" />
-    <origin xyz="0 0 1.15" rpy="0 0 0" />
+    <origin xyz="0 0 1.150" rpy="0 0 0" />
     <axis xyz="0 1 0" />
-    <limit
-      lower="-2.5656"
-      upper="1.5708"
-      effort="0"
-      velocity="2.00713" />
+    <limit lower="${radians(-147)}" upper="${radians(90)}" effort="9806.65" velocity="${radians(115)}" />
   </joint>
   <joint name="${prefix}joint_r" type="revolute">
     <parent link="${prefix}link_u" />
     <child link="${prefix}link_r" />
-    <origin xyz="0.9735 0 0.3" rpy="0 0 0" />
+    <origin xyz="0 0 0.300" rpy="0 0 0" />
     <axis xyz="1 0 0" />
-    <limit
-      lower="-6.2832"
-      upper="6.2832"
-      effort="0"
-      velocity="2.53073" />
+    <limit lower="${radians(-210)}" upper="${radians(210)}" effort="2451.66" velocity="${radians(145)}" />
   </joint>
   <joint name="${prefix}joint_b" type="revolute">
-    <origin xyz="0.2515 0 0" rpy="0 0 0" />
     <parent link="${prefix}link_r" />
     <child link="${prefix}link_b" />
+    <origin xyz="1.225 0 0" rpy="0 0 0" />
     <axis xyz="0 1 0" />
-    <limit
-      lower="-2.2689"
-      upper="2.2689"
-      effort="0"
-      velocity="2.53073" />
+    <limit lower="${radians(-125)}" upper="${radians(125)}" effort="2745.86" velocity="${radians(145)}" />
   </joint>
   <joint name="${prefix}joint_t" type="revolute">
-    <origin xyz="0.21695 0 0" rpy="0 0 0" />
+    <origin xyz="0.250 0 0" rpy="0 0 0" />
     <parent link="${prefix}link_b" />
     <child link="${prefix}link_t" />
     <axis xyz="1 0 0" />
-    <limit
-      lower="-6.2832"
-      upper="6.2832"
-      effort="0"
-      velocity="3.83972" />
+    <limit lower="${radians(-210)}" upper="${radians(210)}" effort="1800.5" velocity="${radians(220)}" />
   </joint>
   <joint name="${prefix}joint_t-tool0" type="fixed">
-    <origin xyz="0.100 0 0 " rpy="0 0 0 "/> <!-- CHECK THIS LINE FOR ACCURACY -->
+    <origin xyz="0 0 0 " rpy="${radians(180)} ${radians(-90)} 0"/>
     <parent link="${prefix}link_t"/>
     <child link="${prefix}tool0"/>
   </joint>
   <!-- end of joint list -->
+  <!-- ROS base_link to Robot Manufacturer World Coordinates transform -->
+  <link name="${prefix}base" />
+  <joint name="${prefix}base_link-base" type="fixed">
+    <origin xyz="0 0 0.650" rpy="0 0 0"/>
+    <parent link="${prefix}base_link"/>
+    <child link="${prefix}base"/>
+  </joint>
   </xacro:macro>
 </robot>
