Commit message: Change MH50 Color name for cluster uniqueness

File: motoman/motoman_mh50_support/urdf/mh50_macro.xacro (robot description, xacro)
@@ -3,5 +3,5 @@
 <xacro:macro name="motoman_mh50" params="prefix">
     <!-- Properties -->
-    <material name="yaskawa_blue">
+    <material name="yaskawa_blue_mh50">
           <color rgba="0.12941 0.14902 0.74902 1" />
     </material>
@@ -12,5 +12,5 @@
                 <mesh filename="package://motoman_mh50_support/meshes/visual/mh50_base_link.stl"/>
             </geometry>
-            <material name="yaskawa_blue"/>
+            <material name="yaskawa_blue_mh50"/>
         </visual>
         <collision>
@@ -25,5 +25,5 @@
                 <mesh filename="package://motoman_mh50_support/meshes/visual/mh50_link_1_s.stl"/>
             </geometry>
-            <material name="yaskawa_blue"/>
+            <material name="yaskawa_blue_mh50"/>
         </visual>
         <collision>
@@ -38,5 +38,5 @@
                 <mesh filename="package://motoman_mh50_support/meshes/visual/mh50_link_2_l.stl"/>
             </geometry>
-            <material name="yaskawa_blue"/>
+            <material name="yaskawa_blue_mh50"/>
         </visual>
         <collision>
@@ -51,5 +51,5 @@
                 <mesh filename="package://motoman_mh50_support/meshes/visual/mh50_link_3_u.stl"/>
             </geometry>
-            <material name="yaskawa_blue"/>
+            <material name="yaskawa_blue_mh50"/>
         </visual>
         <collision>
@@ -64,5 +64,5 @@
                 <mesh filename="package://motoman_mh50_support/meshes/visual/mh50_link_4_r.stl"/>
             </geometry>
-            <material name="yaskawa_blue"/>
+            <material name="yaskawa_blue_mh50"/>
         </visual>
         <collision>
@@ -77,5 +77,5 @@
                 <mesh filename="package://motoman_mh50_support/meshes/visual/mh50_link_5_b.stl"/>
             </geometry>
-            <material name="yaskawa_blue"/>
+            <material name="yaskawa_blue_mh50"/>
         </visual>
         <collision>
@@ -90,5 +90,5 @@
                 <mesh filename="package://motoman_mh50_support/meshes/visual/mh50_link_6_t.stl"/>
             </geometry>
-            <material name="yaskawa_blue"/>
+            <material name="yaskawa_blue_mh50"/>
         </visual>
         <collision>
