Commit message: Add R3 Pick Table

File: core/urdf/environment_macro.xacro (robot description, xacro)
@@ -42,4 +42,18 @@
       <geometry>
         <mesh filename="package://core/meshes/bases/visual/asm_R3_mount_labCoords.STL" />
+      </geometry>
+    </collision>
+  </link>
+  <link  name="${prefix}picktable_r3">
+    <visual>
+      <origin xyz="0 0 -0.889" rpy="0 0 ${radians(180)}" />
+      <geometry>
+        <mesh filename="package://core/meshes/bases/pickTable_R3.STL" />
+      </geometry>
+    </visual>
+    <collision>
+      <origin xyz="0 0 -0.889" rpy="0 0 ${radians(180)}" />
+      <geometry>
+        <mesh filename="package://core/meshes/bases/pickTable_R3.STL" />
       </geometry>
     </collision>
@@ -103,4 +117,9 @@
     <child link="${prefix}mount_r3" />
   </joint>
+  <joint name="${prefix}picktable_r3" type="fixed">
+    <origin xyz="0 0 0" rpy="0 0 0"/>
+    <parent link="${prefix}r3_base_link" />
+    <child link="${prefix}picktable_r3" />
+  </joint>
   <joint name="${prefix}controllerboxes_origin" type="fixed">
     <origin xyz="0 0 0" rpy="0 0 0"/>
