Commit message: Initial Launch Scripts for Cluster

File: core/urdf/cluster_ma2010_ms210_mh50_macro.xacro (robot description, xacro)
@@ -31,5 +31,5 @@
       <xacro:motoman_ms210 prefix="${prefix}r2_"/>
       <joint name="${prefix}r2_joint_origin" type="fixed">
-        <origin xyz="5 0 0" rpy="0 0 0"/>
+        <origin xyz="0 2 0" rpy="0 0 0"/>
         <parent link="${prefix}origin"/>
         <child  link="${prefix}r2_base_link"/>
@@ -37,5 +37,5 @@
       <xacro:motoman_mh50 prefix="${prefix}r3_"/>
       <joint name="${prefix}r3_joint_origin" type="fixed">
-        <origin xyz="10 0 0" rpy="0 0 0"/>
+        <origin xyz=" 0 4 0" rpy="0 0 0"/>
         <parent link="${prefix}origin"/>
         <child  link="${prefix}r3_base_link"/>

Commit message: Add cluster orientation

File: core/urdf/cluster_ma2010_ms210_mh50_macro.xacro (robot description, xacro)
@@ -25,5 +25,5 @@
       <xacro:motoman_ma2010 prefix="${prefix}r1_"/>
       <joint name="${prefix}r1_joint_origin" type="fixed">
-        <origin xyz="0 0 0" rpy="0 0 0"/>
+        <origin xyz="0 0 1.052" rpy="0 0 0"/>
         <parent link="${prefix}origin" />
         <child  link="${prefix}r1_base_link" />
@@ -31,5 +31,5 @@
       <xacro:motoman_ms210 prefix="${prefix}r2_"/>
       <joint name="${prefix}r2_joint_origin" type="fixed">
-        <origin xyz="0 2 0" rpy="0 0 0"/>
+        <origin xyz="0.733 -2.4281 0.127" rpy="0 0 ${radians(90)}"/>
         <parent link="${prefix}origin"/>
         <child  link="${prefix}r2_base_link"/>
@@ -37,5 +37,5 @@
       <xacro:motoman_mh50 prefix="${prefix}r3_"/>
       <joint name="${prefix}r3_joint_origin" type="fixed">
-        <origin xyz=" 0 4 0" rpy="0 0 0"/>
+        <origin xyz="2.03805 -0.66105 0.889" rpy="0 0 ${radians(180)}"/>
         <parent link="${prefix}origin"/>
         <child  link="${prefix}r3_base_link"/>

Commit message: Rollback: Remove EEF & Environment
* Comment out EEF & Environment URDF inclusions.
* Reorganize cluser_macro.xacro

Extra:
* Remove MH5_moveit dependency

File: core/urdf/cluster_ma2010_ms210_mh50_macro.xacro (robot description, xacro)
@@ -3,5 +3,5 @@
   <!-- Properties -->
   <material name="global_yaskawa_blue">
-      <color rgba="0.12941 0.14902 0.74902 1" />
+    <color rgba="0.12941 0.14902 0.74902 1" />
   </material>
   <material name="global_white">
@@ -12,8 +12,4 @@
   <xacro:include filename="$(find motoman_ms210_support)/urdf/ms210_macro.xacro" />
   <xacro:include filename="$(find motoman_mh50_support)/urdf/mh50_macro.xacro" />
-  <!-- Environment -->
-  <xacro:include filename="$(find core)/urdf/environment_macro.xacro" />
-  <!-- End Effectors (EEF) -->
-  <xacro:include filename="$(find core)/urdf/endeffectors_macro.xacro" />
   <!-- Robot Cluster Definition -->
   <xacro:macro name="cluster_ma2010_ms210_mh50" params="prefix">
@@ -45,7 +41,12 @@
         <child  link="${prefix}r3_base_link"/>
       </joint>
+      <!-- Environment -->
+  <!--<xacro:include filename="$(find core)/urdf/environment_macro.xacro" />
       <xacro:aims_environment prefix="${prefix}"/>
+  -->
+      <!-- End Effectors (EEF) -->
+  <!--<xacro:include filename="$(find core)/urdf/endeffectors_macro.xacro" />
       <xacro:cluster_eef prefix="${prefix}"/>
+  -->
   </xacro:macro>
-  <!-- Robot Cluster Inclusion -->
 </robot>

File: core/urdf/endeffectors_macro.xacro (robot description, xacro)
@@ -2,44 +2,44 @@
 <robot xmlns:xacro="http://ros.org/wiki/xacro">
 <xacro:macro name="cluster_eef" params="prefix">
-  <!-- Link List -->
-<link  name="${prefix}eef_r2">
-  <visual>
-    <origin xyz="0 0 0" rpy="0 0 0" />
-    <geometry>
-      <mesh filename="package://core/meshes/eef/r2_approx.stl" />
-    </geometry>
-  </visual>
-  <collision>
-    <origin xyz="0 0 0" rpy="0 0 0" />
-    <geometry>
-      <mesh filename="package://core/meshes/eef/r2_approx.stl" />
-    </geometry>
-  </collision>
-</link>
-<link  name="${prefix}eef_r3">
-  <visual>
-    <origin xyz="0 0 0" rpy="0 0 0" />
-    <geometry>
-      <mesh filename="package://core/meshes/eef/r3_approx.stl" />
-    </geometry>
-  </visual>
-  <collision>
-    <origin xyz="0 0 0" rpy="0 0 0" />
-    <geometry>
-      <mesh filename="package://core/meshes/eef/r3_approx.stl" />
-    </geometry>
-  </collision>
-</link>
-<!-- Joint List -->
-<joint name="${prefix}eef_r2_tool0" type="fixed">
-  <origin xyz="0 0 0" rpy="0 0 0"/>
-  <parent link="${prefix}r2_tool0" />
-  <child link="${prefix}eef_r2" />
-</joint>
-<joint name="${prefix}eef_r3_tool0" type="fixed">
-  <origin xyz="0 0 0.03" rpy="${radians(-90)} 0 0"/>
-  <parent link="${prefix}r3_tool0" />
-  <child link="${prefix}eef_r3" />
-</joint>
+  <!-- R2 EEF -->
+  <link  name="${prefix}eef_r2">
+    <visual>
+      <origin xyz="0 0 0" rpy="0 0 0" />
+      <geometry>
+        <mesh filename="package://core/meshes/eef/r2_approx.stl" />
+      </geometry>
+    </visual>
+    <collision>
+      <origin xyz="0 0 0" rpy="0 0 0" />
+      <geometry>
+        <mesh filename="package://core/meshes/eef/r2_approx.stl" />
+      </geometry>
+    </collision>
+  </link>
+  <joint name="${prefix}eef_r2_tool0" type="fixed">
+    <origin xyz="0 0 0" rpy="0 0 0"/>
+    <parent link="${prefix}r2_tool0" />
+    <child link="${prefix}eef_r2" />
+  </joint>
+  <!-- R3 EEF -->
+  <link  name="${prefix}eef_r3">
+    <visual>
+      <origin xyz="0 0 0" rpy="0 0 0" />
+      <geometry>
+        <mesh filename="package://core/meshes/eef/r3_approx.stl" />
+      </geometry>
+    </visual>
+    <collision>
+      <origin xyz="0 0 0" rpy="0 0 0" />
+      <geometry>
+        <mesh filename="package://core/meshes/eef/r3_approx.stl" />
+      </geometry>
+    </collision>
+    <joint name="${prefix}eef_r3_tool0" type="fixed">
+      <origin xyz="0 0 0.03" rpy="${radians(-90)} 0 0"/>
+      <parent link="${prefix}r3_tool0" />
+      <child link="${prefix}eef_r3" />
+    </joint>
+  </link>
 </xacro:macro>
 </robot>
