Commit message: Dev - Integrate Envir Package & Misc Updates
- fixed cognex camera rotation
- updated moveit predefined collisions using setup assistant.
- simplify pick table collision mesh to convex hulls
- switched global origin to be defined by CORE package and not 
environment package.

File: aims_environment/urdf/environment.xacro (robot description, xacro)
@@ -3,4 +3,5 @@
 	<xacro:include filename="$(find aims_environment)/urdf/environment_macro.xacro" />
 	<xacro:aims_environment prefix=""/>
+<!--
   <link name="origin_global">
     <visual>
@@ -12,3 +13,4 @@
     </visual>
   </link>
+-->
 </robot>

File: aims_environment/urdf/environment_macro.xacro (robot description, xacro)
@@ -166,5 +166,5 @@
   </joint>
   <joint name="${prefix}cognex_origin" type="fixed">
-    <origin xyz="1 -0.7 3.2" rpy="0 0 ${radians(90)}"/>
+    <origin xyz="1 -0.7 3.2" rpy="0 0 ${radians(180)}"/>
     <parent link="origin_global" />
     <child link="${prefix}cognex" />

File: core/urdf/cluster_ma2010_ms210_mh50_macro.xacro (robot description, xacro)
@@ -13,10 +13,10 @@
   <xacro:include filename="$(find motoman_mh50_support)/urdf/mh50_macro.xacro" />
   <!-- Environment -->
-  <xacro:include filename="$(find core)/urdf/environment_macro.xacro" />
+  <xacro:include filename="$(find aims_environment)/urdf/environment_macro.xacro" />
   <!-- End Effectors (EEF) -->
   <xacro:include filename="$(find core)/urdf/endeffectors_macro.xacro" />
   <!-- Robot Cluster Definition -->
   <xacro:macro name="cluster_ma2010_ms210_mh50" params="prefix">
-      <link name="${prefix}origin">
+      <link name="${prefix}origin_global">
         <visual>
           <origin xyz="0 0 0" rpy="0 0 0" />
@@ -30,5 +30,5 @@
       <joint name="${prefix}r1_joint_origin" type="fixed">
         <origin xyz="0 0 1.052" rpy="0 0 0"/>
-        <parent link="${prefix}origin" />
+        <parent link="${prefix}origin_global" />
         <child  link="${prefix}r1_base_link" />
       </joint>
@@ -36,5 +36,5 @@
       <joint name="${prefix}r2_joint_origin" type="fixed">
         <origin xyz="0.733 -2.4281 0.127" rpy="0 0 ${radians(90)}"/>
-        <parent link="${prefix}origin"/>
+        <parent link="${prefix}origin_global"/>
         <child  link="${prefix}r2_base_link"/>
       </joint>
@@ -42,5 +42,5 @@
       <joint name="${prefix}r3_joint_origin" type="fixed">
         <origin xyz="2.03805 -0.66105 0.889" rpy="0 0 ${radians(180)}"/>
-        <parent link="${prefix}origin"/>
+        <parent link="${prefix}origin_global"/>
         <child  link="${prefix}r3_base_link"/>
       </joint>
