Commit message: Mass Rewrite & Restructure of support package
* rename from `core` to `aims_wc1_support` to better reflect intention of package
* remove scraps

Still includes bloat mesh files and incomplete environment URDF.

File: aims_wc1_support/urdf/endeffectors_macro.xacro (robot description, xacro)
@@ -7,5 +7,5 @@
       <origin xyz="0 0 0" rpy="0 0 0" />
       <geometry>
-        <mesh filename="package://core/meshes/eef/r2_approx.stl" />
+        <mesh filename="package://aims_wc1_support/meshes/eef/r2_approx.stl" />
       </geometry>
     </visual>
@@ -13,5 +13,5 @@
       <origin xyz="0 0 0" rpy="0 0 0" />
       <geometry>
-        <mesh filename="package://core/meshes/eef/r2_approx.stl" />
+        <mesh filename="package://aims_wc1_support/meshes/eef/r2_approx.stl" />
       </geometry>
     </collision>
@@ -27,5 +27,5 @@
       <origin xyz="0 0 0" rpy="0 0 0" />
       <geometry>
-        <mesh filename="package://core/meshes/eef/r3_approx.stl" />
+        <mesh filename="package://aims_wc1_support/meshes/eef/r3_approx.stl" />
       </geometry>
     </visual>
@@ -33,5 +33,5 @@
       <origin xyz="0 0 0" rpy="0 0 0" />
       <geometry>
-        <mesh filename="package://core/meshes/eef/r3_approx.stl" />
+        <mesh filename="package://aims_wc1_support/meshes/eef/r3_approx.stl" />
       </geometry>
     </collision>

File: aims_wc1_support/urdf/environment_macro.xacro (robot description, xacro)
@@ -7,5 +7,5 @@
       <origin xyz="0 0 -1.051999" rpy="0 0 0" />
       <geometry>
-        <mesh filename="package://core/meshes/bases/visual/asm_R1_mount_labCoords.STL" />
+        <mesh filename="package://aims_wc1_support/meshes/bases/visual/asm_R1_mount_labCoords.STL" />
       </geometry>
     </visual>
@@ -13,5 +13,5 @@
       <origin xyz="0 0 -1.051999" rpy="0 0 0" />
       <geometry>
-        <mesh filename="package://core/meshes/bases/visual/asm_R1_mount_labCoords.STL" />
+        <mesh filename="package://aims_wc1_support/meshes/bases/visual/asm_R1_mount_labCoords.STL" />
       </geometry>
     </collision>
@@ -21,5 +21,5 @@
       <origin xyz="0 0 -.127" rpy="0 0 ${radians(-90)}" />
       <geometry>
-        <mesh filename="package://core/meshes/bases/visual/asm_R2_mount_labCoords.STL" />
+        <mesh filename="package://aims_wc1_support/meshes/bases/visual/asm_R2_mount_labCoords.STL" />
       </geometry>
     </visual>
@@ -27,5 +27,5 @@
       <origin xyz="0 0 -.127" rpy="0 0 ${radians(-90)}" />
       <geometry>
-        <mesh filename="package://core/meshes/bases/visual/asm_R2_mount_labCoords.STL" />
+        <mesh filename="package://aims_wc1_support/meshes/bases/visual/asm_R2_mount_labCoords.STL" />
       </geometry>
     </collision>
@@ -35,5 +35,5 @@
       <origin xyz="0 0 -0.889" rpy="${radians(90)} 0 0" />
       <geometry>
-        <mesh filename="package://core/meshes/bases/visual/asm_R3_mount_labCoords.STL" />
+        <mesh filename="package://aims_wc1_support/meshes/bases/visual/asm_R3_mount_labCoords.STL" />
       </geometry>
     </visual>
@@ -41,5 +41,5 @@
       <origin xyz="0 0 -0.889" rpy="${radians(90)} 0 0" />
       <geometry>
-        <mesh filename="package://core/meshes/bases/visual/asm_R3_mount_labCoords.STL" />
+        <mesh filename="package://aims_wc1_support/meshes/bases/visual/asm_R3_mount_labCoords.STL" />
       </geometry>
     </collision>
@@ -49,5 +49,5 @@
       <origin xyz="0 0 -0.889" rpy="0 0 ${radians(180)}" />
       <geometry>
-        <mesh filename="package://core/meshes/bases/pickTable_R3.STL" />
+        <mesh filename="package://aims_wc1_support/meshes/bases/pickTable_R3.STL" />
       </geometry>
     </visual>
@@ -55,5 +55,5 @@
       <origin xyz="0 0 -0.889" rpy="0 0 ${radians(180)}" />
       <geometry>
-        <mesh filename="package://core/meshes/bases/pickTable_R3.STL" />
+        <mesh filename="package://aims_wc1_support/meshes/bases/pickTable_R3.STL" />
       </geometry>
     </collision>
@@ -63,5 +63,5 @@
       <origin xyz="-1 -0.8 0" rpy="0 0 0" />
       <geometry>
-        <mesh filename="package://core/meshes/equipment/dx200_controller_boxes.STL" />
+        <mesh filename="package://aims_wc1_support/meshes/equipment/dx200_controller_boxes.STL" />
       </geometry>
     </visual>
@@ -69,5 +69,5 @@
       <origin xyz="0 0 -0.889" rpy="0 0 0" />
       <geometry>
-        <mesh filename="package://core/meshes/equipment/dx200_controller_boxes.STL" />
+        <mesh filename="package://aims_wc1_support/meshes/equipment/dx200_controller_boxes.STL" />
       </geometry>
     </collision>
@@ -77,5 +77,5 @@
       <origin xyz="0 -4 0" rpy="0 0 0" />
       <geometry>
-        <mesh filename="package://core/meshes/equipment/tormach_mill_rough.STL" />
+        <mesh filename="package://aims_wc1_support/meshes/equipment/tormach_mill_rough.STL" />
       </geometry>
     </visual>
@@ -83,5 +83,5 @@
       <origin xyz="0 -4 0" rpy="0 0 0" />
       <geometry>
-        <mesh filename="package://core/meshes/equipment/tormach_mill_rough.STL" />
+        <mesh filename="package://aims_wc1_support/meshes/equipment/tormach_mill_rough.STL" />
       </geometry>
     </collision>
@@ -91,5 +91,5 @@
       <origin xyz="1 -0.7 3.2" rpy="0 0 0" />
       <geometry>
-        <mesh filename="package://core/meshes/equipment/cognex_ceiling_assembly.STL" />
+        <mesh filename="package://aims_wc1_support/meshes/equipment/cognex_ceiling_assembly.STL" />
       </geometry>
     </visual>
@@ -97,5 +97,5 @@
       <origin xyz="1 -0.7 3.2" rpy="0 0 0" />
       <geometry>
-        <mesh filename="package://core/meshes/equipment/cognex_ceiling_assembly.STL" />
+        <mesh filename="package://aims_wc1_support/meshes/equipment/cognex_ceiling_assembly.STL" />
       </geometry>
     </collision>
